File: projects/SafeWalk/Schema 3.sch (EAGLE design)
At the start: 18 parts

Commit message: board 1
Parts:
- removed J_ULTRASONIC_3, J_ULTRASONIC_4: HC-SR04, Ultrasonic Sensor HC-SR04:HC-SR04
- removed SG2: EB2505, buzzer:EB2505
- removed SV1, SV2: (no value), con-lsta:FE15-1
- removed X5, X6, X7, X8, X9: (no value), con-ptr500:AK300/2
Connections:
- removed net N$11: J_ULTRASONIC_3.ECHO, SV2.3, X5-2.KL
- removed net N$12: J_ULTRASONIC_4.TRIG, SV2.4, X6-1.KL
- removed net N$13: J_ULTRASONIC_4.ECHO, SV2.5, X6-2.KL, X7-2.KL
- removed net N$14: SG2.+, SV2.7, X7-1.KL
- removed net N$15: J_ULTRASONIC_3.5V, SV2.15, X8-2.KL
- removed net N$16: J_ULTRASONIC_3.GND, X8-1.KL
- removed net N$17: J_ULTRASONIC_4.GND, SG2.-, SV1.2, X9-1.KL
- removed net N$18: J_ULTRASONIC_4.5V, SV1.5
- removed net N$19: SV1.1, X9-2.KL
- removed net N$20: SV2.14
- removed net N$5: J_ULTRASONIC_3.TRIG, SV2.2, X5-1.KL
