File: projects/SafeWalk/Schema 6.brd (EAGLE design)
At the start: 100 x 80 mm, 6 parts

Commit message: upload malam ini
Parts:
- moved X1 8.85 mm to (57.1, 59.8)
- moved J_ULTRASONIC_4 5.10 mm to (22.3, 38.1)
- moved SG2 5.02 mm to (80.3, 63.3)
- moved J_ULTRASONIC_3 3.83 mm to (22.2, 20.3)
- moved SV2 1.02 mm to (74.5, 42.0)
- moved SV1 1.00 mm to (74.5, 14.1)
Routing:
- net N$8: track 112.7 -> 0.00 mm
- net N$9: track 101.5 -> 0.00 mm
- net N$5: track 137.2 -> 119.1 mm
- net N$6: track 45.9 -> 31.7 mm
- net N$4: track 44.0 -> 36.1 mm
- net N$7: track 67.5 -> 71.5 mm
- net N$10: track 55.0 -> 52.6 mm
- net N$2: track 67.8 -> 69.6 mm
- net N$1: track 72.3 -> 73.6 mm
- net N$3: track 58.7 -> 57.6 mm
Other:
- board text removed: "+"
- board text removed: "-"
- board text removed: "Battery"
- board text removed: "Buzzer"
- board text removed: "D0"
- board text removed: "D1"
- board text removed: "D2"
- board text removed: "ECHO"
- board text removed: "ESP8266"
- board text removed: "GND"
- board text removed: "Safewalk Projet Danes-Aul-Bijak-Adzima-Genta Della-Kaysa-Kevin-Memed"
- board text removed: "Sensor 1"
- board text removed: "Sensor 2"
- board text removed: "TRIGGER"
- board text removed: "VCC"

Commit message: GPS done laptop Adzima
Routing:
- net N$8: track 0.00 -> 116.1 mm
- net N$9: track 0.00 -> 103.1 mm
- added copper zone on layer 16, net TST
Changed lines of the file:
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@@
 </class>
 </classes>
-<designrules name="default">
+<designrules name="default *">
 <description language="de">&lt;b&gt;EAGLE Design Rules&lt;/b&gt;
 &lt;p&gt;
@@
 <param name="mtCopper" value="0.035mm 0.035mm 0.035mm 0.035mm 0.035mm 0.035mm 0.035mm 0.035mm 0.035mm 0.035mm 0.035mm 0.035mm 0.035mm 0.035mm 0.035mm 0.035mm"/>
 <param name="mtIsolate" value="1.5mm 0.15mm 0.2mm 0.15mm 0.2mm 0.15mm 0.2mm 0.15mm 0.2mm 0.15mm 0.2mm 0.15mm 0.2mm 0.15mm 0.2mm"/>
-<param name="mdWireWire" value="6mil"/>
-<param name="mdWirePad" value="6mil"/>
-<param name="mdWireVia" value="6mil"/>
-<param name="mdPadPad" value="6mil"/>
-<param name="mdPadVia" value="6mil"/>
-<param name="mdViaVia" value="6mil"/>
-<param name="mdSmdPad" value="6mil"/>
-<param name="mdSmdVia" value="6mil"/>
-<param name="mdSmdSmd" value="6mil"/>
+<param name="mdWireWire" value="40mil"/>
+<param name="mdWirePad" value="40mil"/>
+<param name="mdWireVia" value="40mil"/>
+<param name="mdPadPad" value="40mil"/>
+<param name="mdPadVia" value="40mil"/>
+<param name="mdViaVia" value="40mil"/>
+<param name="mdSmdPad" value="40mil"/>
+<param name="mdSmdVia" value="40mil"/>
+<param name="mdSmdSmd" value="40mil"/>
 <param name="mdViaViaSameLayer" value="6mil"/>
 <param name="mnLayersViaInSmd" value="2"/>
@@
 <contactref element="J_ULTRASONIC_4" pad="ECHO"/>
 <contactref element="SV1" pad="12"/>
-<wire x1="22.343" y1="39.338" x2="84.696" y2="14.104" width="0" layer="19" extent="1-1"/>
+<wire x1="22.343" y1="39.338" x2="16.097" y2="39.338" width="0.8128" layer="16"/>
+<wire x1="16.097" y1="39.338" x2="11.811" y2="35.052" width="0.8128" layer="16"/>
+<wire x1="11.811" y1="35.052" x2="11.811" y2="12.446" width="0.8128" layer="16"/>
+<wire x1="11.811" y1="12.446" x2="18.288" y2="5.969" width="0.8128" layer="16"/>
+<wire x1="80.391" y1="5.969" x2="18.288" y2="5.969" width="0.8128" layer="16"/>
+<wire x1="84.696" y1="14.104" x2="84.696" y2="10.274" width="0.8128" layer="16"/>
+<wire x1="84.696" y1="10.274" x2="80.391" y2="5.969" width="0.8128" layer="16"/>
 </signal>
 <signal name="N$9">
 <contactref element="J_ULTRASONIC_4" pad="TRIG"/>
 <contactref element="SV1" pad="11"/>
-<wire x1="22.343" y1="36.798" x2="82.156" y2="14.104" width="0" layer="19" extent="1-1"/>
+<wire x1="22.343" y1="36.798" x2="17.24" y2="36.798" width="0.8128" layer="16"/>
+<wire x1="17.24" y1="36.798" x2="14.478" y2="34.036" width="0.8128" layer="16"/>
+<wire x1="14.478" y1="34.036" x2="14.478" y2="13.522" width="0.8128" layer="16"/>
+<wire x1="14.478" y1="13.522" x2="19.397" y2="8.603" width="0.8128" layer="16"/>
+<wire x1="19.397" y1="8.603" x2="79.342" y2="8.603" width="0.8128" layer="16"/>
+<wire x1="82.156" y1="11.417" x2="82.156" y2="14.104" width="0.8128" layer="16"/>
+<wire x1="79.342" y1="8.603" x2="82.156" y2="11.417" width="0.8128" layer="16"/>
+</signal>
+<signal name="TST">
+<polygon width="1.016" layer="16">
+<vertex x="0" y="80"/>
+<vertex x="0" y="0"/>
+<vertex x="100" y="0"/>
+<vertex x="100" y="80"/>
+</polygon>
 </signal>
 </signals>
@@
 <mfgpreviewcolor name="substratecolor" color="0xFF786E46"/>
 </mfgpreviewcolors>
+<errors>
+</errors>
 </board>
 </drawing>
