File: projects/SafeWalk/With GPS.brd (EAGLE design)
At the start: 100 x 80 mm, 6 parts

Commit message: GPS done laptop Adzima
Parts:
- added X2: (no value), con-ptr500:AK300/4
- moved X1 10.2 mm to (51.3, 68.2)
- moved J_ULTRASONIC_3 4.57 mm to (26.0, 17.8)
- moved J_ULTRASONIC_4 3.93 mm to (26.0, 39.6), turned to 180 degrees
- moved SV1 3.62 mm to (71.0, 14.7)
- moved SV2 3.57 mm to (71.0, 42.7)
- moved SG2 3.22 mm to (83.3, 62.2), turned to 90 degrees
Connections:
- removed net N$5: J_ULTRASONIC_4.GND, SG2.-, SV2.14, X1.1
- new net N$11: SV1.8, X2.3
- new net N$12: SV1.7, X2.2
- new net N$13: J_ULTRASONIC_4.GND, SG2.-, SV2.14, X1.1, X2.1
- net N$10: now also X2.4
Routing:
- net N$13: track 0.00 -> 244.3 mm
- net N$12: track 0.00 -> 146.8 mm
- net N$11: track 0.00 -> 133.1 mm
- net N$5: track 119.1 -> 0.00 mm
- net N$9: track 0.00 -> 94.4 mm
- net N$8: track 0.00 -> 88.0 mm
- net N$1: track 73.6 -> 106.5 mm
- net N$10: track 52.6 -> 78.9 mm
- net N$3: track 57.6 -> 35.2 mm
- net N$2: track 69.6 -> 90.9 mm
- net N$7: track 71.5 -> 52.5 mm
- net N$4: track 36.1 -> 29.1 mm
- net N$6: track 31.7 -> 27.3 mm
- added copper zone on layer 16, net 1
Other:
- board text added: "BUZZER"
- board text added: "ESP KANAN"
- board text added: "ESP KIRI"
- board text added: "GPS MODULE"
- board text added: "SENSOR 1"
- board text added: "SENSOR 2"
